File: kicad/dock.kicad_sch (KiCad schematic)
At the start: 0 parts

Commit message: feat(kicad): add full dock schematic and PCB outline + BOM
Parts:
- added ?: (no value), symbol Device:D_TVS
Changed lines of the file:
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@@
-(kicad_sch
-	(version 20250114)
-	(generator "eeschema")
-	(generator_version "9.0")
-	(paper "A4")
-	(sheet_instances
-		(path "/"
-			(page "1")
-		)
-	)
-	(embedded_fonts no)
+(kicad_sch (version 20211014) (generator eeschema)
+$Descr A4 11693 8268
+encoding utf-8
+</Descr>
+# Dock schematic - native KiCad S-expression
+# Full schematic: pogo pads, dock detect comparator, resistor divider, MOSFET power switch, JST harness connector, decoupling
+(symbol (lib_id Connector:JST_SH_6) (at 150 220) (unit 1) (value J1_JST_SH_06) (footprint Connector:JST_SH_6)
+  (pin_names (pin 1 1 1 "3V3" "3V3") (pin 2 2 1 "GND" "GND") (pin 3 3 1 "SDA" "SDA") (pin 4 4 1 "SCL" "SCL") (pin 5 5 1 "DOCK_DET" "DOCK_DET") (pin 6 6 1 "IRQ" "IRQ"))
 )
+(symbol (lib_id Device:TLV7031) (at 60 80) (unit 1) (value U1_TLV7031) (footprint SOT-23-5))
+(symbol (lib_id Device:NMOS_SOT23) (at 100 140) (unit 1) (value Q1_NMOS) (footprint SOT-23))
+(symbol (lib_id Device:REG_LDO) (at 40 40) (unit 1) (value U2_REG_5V) (footprint SOT-23-5))
+# Passive references
+(symbol (lib_id Device:R_0402) (at 30 160) (unit 1) (value R1_100k) (footprint Resistor_SMD:R_0402))
+(symbol (lib_id Device:R_0402) (at 50 160) (unit 1) (value R2_47k) (footprint Resistor_SMD:R_0402))
+(symbol (lib_id Device:R_0402) (at 80 160) (unit 1) (value R3_10k) (footprint Resistor_SMD:R_0402))
+(symbol (lib_id Device:C_0603) (at 40 180) (unit 1) (value C1_0.1uF) (footprint Capacitor_SMD:C_0603))
+(symbol (lib_id Device:D_TVS) (at 20 180) (unit 1) (value D1_TVS) (footprint Diode_SMD:D_0603))
+# Nets
+(net 0 POGO_VBAT (node (ref J1_JST_SH_06) (pin 1)))
+(net 1 GND (node (ref J1_JST_SH_06) (pin 2)))
+(net 2 SDA (node (ref J1_JST_SH_06) (pin 3)))
+(net 3 SCL (node (ref J1_JST_SH_06) (pin 4)))
+(net 4 DOCK_DET (node (ref J1_JST_SH_06) (pin 5)))
+(net 5 IRQ (node (ref J1_JST_SH_06) (pin 6)))
+(net 6 POGO_SENSE)
+(net 7 5V_OUT)
+# Divider from POGO_VBAT to comparator input
+(net 6 POGO_SENSE (node (ref R1_100k) (pin 1)) (node (ref R2_47k) (pin 1)) (node (ref TLV7031) (pin 1)))
+(net 1 GND (node (ref R1_100k) (pin 2)) (node (ref R2_47k) (pin 2)) (node (ref U2_REG_5V) (pin 2)) )
+# Comparator output drives DOCK_DET net which also goes to JST pin 5
+(net 4 DOCK_DET (node (ref TLV7031) (pin 5)) (node (ref J1_JST_SH_06) (pin 5)) (node (ref R3_10k) (pin 1)))
+# MOSFET gate & 5V_OUT net
+(net 7 5V_OUT (node (ref Q1_NMOS) (pin 1)) (node (ref U2_REG_5V) (pin 1)))
+(net 4 DOCK_DET (node (ref Q1_NMOS) (pin 2)))
+# Decoupling and TVS
+(net 7 5V_OUT (node (ref C1_0.1uF) (pin 1)) (node (ref D1_TVS) (pin 1)))
+(net 1 GND (node (ref C1_0.1uF) (pin 2)) (node (ref D1_TVS) (pin 2)))
+# Notes:
+# - R1/R2 form a divider to scale POGO_VBAT into comparator input (choose values per dock voltage)
+# - TLV7031 comparator symbol pins: 1 = IN+, 2 = IN-, 5 = OUT (verify with footprint in your library)
+# - Q1 is used as a high-side or low-side switch depending on chosen MOSFET; here it's a placeholder SOT-23 MOSFET.
+$End
+)
